Commit message: SImulation of apostile_robot in gazebo

File: urdf/custom_bot.urdf (robot description, URDF)
Before this commit: robot apostile_robot, 6 links, 5 joints
Links:
- link back_left_wheel: mass None -> 0.6; geometry collision cylinder length=0.025 radius=0.06; visual cylinder length=0.025 radius=0.06
- link back_right_wheel: mass None -> 0.6; geometry collision cylinder length=0.025 radius=0.06; visual cylinder length=0.025 radius=0.06
- link base_link: mass None -> 5.6; geometry collision box size=0.366 0.2934 0.136; visual box size=0.366 0.2934 0.136
- link front_left_wheel: mass None -> 0.6; geometry collision cylinder length=0.025 radius=0.06; visual cylinder length=0.025 radius=0.06
- link front_right_wheel: mass None -> 0.6; geometry collision cylinder length=0.025 radius=0.06; visual cylinder length=0.025 radius=0.06
- link lidar: geometry collision cylinder length=0.055 radius=0.035; visual cylinder length=0.055 radius=0.035

Commit message: generated map via rviz

File: urdf/custom_bot.urdf (robot description, URDF)
Before this commit: robot apostile_robot, 6 links, 5 joints
Links:
- removed link base_link
- added link Robot_base, mass 5.6; collision box size=0.366 0.2934 0.136; visual box size=0.366 0.2934 0.136
Joints:
- joint back_left_wheel_joint: parent base_link -> Robot_base
- joint back_right_wheel_joint: parent base_link -> Robot_base
- joint front_left_wheel_joint: parent base_link -> Robot_base
- joint front_right_wheel_joint: parent base_link -> Robot_base
- joint lidar_joint: parent base_link -> Robot_base
